Commit message: updated robot description with inertia and diff drive plugins

File: description/robot_core.xacro (robot description, xacro)
@@ -42,4 +42,7 @@
         </xacro:inertial_box>
     </link>
+    <gazebo reference="chassis">
+        <material>Gazebo/White</material>
+    </gazebo>
     <!-- LEFT WHEEL LINK -->
     <joint name = "left_wheel_joint" type="continuous">
@@ -65,4 +68,7 @@
         </xacro:inertial_cylinder>
     </link>
+    <gazebo reference="left_wheel">
+        <material>Gazebo/Blue</material>
+    </gazebo>
     <!-- RIGHT WHEEL LINK -->
     <joint name = "right_wheel_joint" type="continuous">
@@ -88,4 +94,7 @@
         </xacro:inertial_cylinder>
     </link>
+    <gazebo reference="right_wheel">
+        <material>Gazebo/Blue</material>
+    </gazebo>
     <!-- CASTER WHEEL LINK -->
     <joint name="caster_wheel_joint" type="fixed">
@@ -110,3 +119,8 @@
         </xacro:inertial_sphere>
     </link>
+    <gazebo reference="caster_wheel">
+        <material>Gazebo/Black</material>
+        <mu1 value="0.001"/>
+        <mu2 value="0.001"/>
+    </gazebo>
 </robot>

Commit message: updated wheel position

File: description/robot_core.xacro (robot description, xacro)
@@ -49,5 +49,5 @@
         <parent link="base_link"/>
         <child link = "left_wheel"/>
-        <origin xyz="0 0.1 -0.035" rpy="-${pi/2} 0 0"/> <!-- The left wheel is 0.1m left and 0.035m below the base link origin, and rotated to be on its side-->
+        <origin xyz="0 0.095 -0.035" rpy="-${pi/2} 0 0"/> <!-- The left wheel is 0.1m left and 0.035m below the base link origin, and rotated to be on its side-->
         <axis xyz="0 0 1"/> <!-- Forward rotation is positive around z axis-->
     </joint>

Commit message: added green colour

File: description/robot_core.xacro (robot description, xacro)
@@ -13,4 +13,7 @@
     <material name="black">
         <color rgba="0 0 0 1"/>
+    </material>
+    <material name="green">
+        <color rgba="0 1 0 1"/>
     </material>
     <!-- BASE LINK-->

Commit message: roboto model uses spheres for collision on wheels to reduce friction

File: description/robot_core.xacro (robot description, xacro)
@@ -64,5 +64,5 @@
         <collision>
             <geometry>
-                <cylinder radius="0.034" length="0.025"/>
+                <sphere radius="0.034"/>
             </geometry>
         </collision>
@@ -90,5 +90,5 @@
         <collision>
             <geometry>
-                <cylinder radius="0.034" length="0.025"/>
+                <sphere radius="0.034"/>
             </geometry>
         </collision>

Commit message: added base footprint

File: description/robot_core.xacro (robot description, xacro)
@@ -20,4 +20,12 @@
     <!-- base link origin centre point between two wheels -->
     <link name="base_link">
+    </link>
+    <!-- BASE_FOOTPRINT LINK -->
+    <joint name="base_footprint_joint" type="fixed">
+        <parent link="base_link"/>
+        <child link="base_footprint"/>
+        <origin xyz="0 0 0" rpy="0 0 0"/>
+    </joint>
+    <link name="base_footprint">
     </link>
     <!-- CHASSIS LINK -->
